Commit message: gazebo not move

File: src/model/xacro/gazebo/base.xacro (robot description, xacro)
@@ -1,11 +1,14 @@
 <robot name="model" xmlns:xacro="http://wiki.ros.org/xacro">
-    <gazebo reference="left_wheel">
+    <gazebo reference="l_wheel">
         <material>Gazebo/Black</material>
     </gazebo>
-    <gazebo reference="right_wheel">
+    <gazebo reference="r_wheel">
         <material>Gazebo/Black</material>
     </gazebo>
-    <gazebo reference="back_wheel">
+    <gazebo reference="b_wheel">
         <material>Gazebo/Black</material>
+    </gazebo>
+    <gazebo reference="f_wheel">
+        <material>Gazebo/Read</material>
     </gazebo>
     <gazebo reference="base_link">
@@ -13,12 +16,12 @@
     </gazebo>
         <!-- 传动实现:用于连接控制器与关节 -->
-    <xacro:macro name="joint_transmission" params="joint_name">
+    <xacro:macro name="joint_transmission" params="wheel_name">
         <!-- Transmission is important to link the joints and the controller -->
-        <transmission name="${joint_name}_transmission">
+        <transmission name="${wheel_name}_transmission">
             <type>transmission_interface/SimpleTransmission</type>
-            <joint name="${joint_name}">
+            <joint name="${wheel_name}_joint">
                 <hardwareInterface>hardware_interface/VelocityJointInterface</hardwareInterface>
             </joint>
-            <actuator name="${joint_name}_motor">
+            <actuator name="${wheel_name}_motor">
                 <hardwareInterface>hardware_interface/VelocityJointInterface</hardwareInterface>
                 <mechanicalReduction>1</mechanicalReduction>
@@ -27,6 +30,6 @@
     </xacro:macro>
     <!-- 每一个驱动轮都需要配置传动装置 -->
-    <xacro:joint_transmission joint_name="left_joint" />
-    <xacro:joint_transmission joint_name="right_joint" />
+    <xacro:joint_transmission wheel_name="l_wheel"/>
+    <xacro:joint_transmission wheel_name="r_wheel"/>
     <!-- 控制器 -->
     <gazebo>
@@ -40,8 +43,8 @@
             <updateRate>100.0</updateRate>
             <legacyMode>true</legacyMode>
-            <leftJoint>left_joint</leftJoint> <!-- 左轮 -->
-            <rightJoint>right_joint</rightJoint> <!-- 右轮 -->
-            <wheelSeparation>${wheel_between}</wheelSeparation> <!-- 车轮间距 -->
-            <wheelDiameter>${wheel_radius * 2}</wheelDiameter> <!-- 车轮直径 -->
+            <leftJoint>l_wheel_joint</leftJoint> <!-- 左轮 -->
+            <rightJoint>r_wheel_joint</rightJoint> <!-- 右轮 -->
+            <wheelSeparation>${wheel_driving_between}</wheelSeparation> <!-- 车轮间距 -->
+            <wheelDiameter>${wheel_driving_radius * 2}</wheelDiameter> <!-- 车轮直径 -->
             <broadcastTF>1</broadcastTF>
             <wheelTorque>30</wheelTorque>
@@ -50,4 +53,6 @@
             <odometryFrame>odom</odometryFrame>
             <odometryTopic>odom</odometryTopic> <!-- 里程计话题 -->
+            <odometrySource>1</odometrySource>
+            <publishOdomTF>true</publishOdomTF>
             <robotBaseFrame>base_footprint</robotBaseFrame> <!-- 根坐标系 -->
         </plugin>

File: src/model/xacro/link/robot.xacro (robot description, xacro)
@@ -1,10 +1,9 @@
 <robot name="robot" xmlns:xacro="http://wiki.ros.org/xacro">
+    <!--xacro-->
     <xacro:include filename="ineritial.xacro"/>
     <xacro:include filename="base.xacro"/>
     <xacro:include filename="laser.xacro"/>
     <!--gazebo仿真-->
-    <!--
     <xacro:include filename="../gazebo/base.xacro"/>
     <xacro:include filename="../gazebo/laser.xacro"/>
-    -->
 </robot>

Commit message: server for amcl navigation

File: src/model/xacro/gazebo/base.xacro (robot description, xacro)
@@ -20,5 +20,5 @@
         <transmission name="${wheel_name}_transmission">
             <type>transmission_interface/SimpleTransmission</type>
-            <joint name="${wheel_name}_joint">
+            <joint name="base_${wheel_name}_joint">
                 <hardwareInterface>hardware_interface/VelocityJointInterface</hardwareInterface>
             </joint>
@@ -41,8 +41,8 @@
             <publishWheelJointState>true</publishWheelJointState>
             <alwaysOn>true</alwaysOn>
-            <updateRate>100.0</updateRate>
+            <updateRate>150.0</updateRate>
             <legacyMode>true</legacyMode>
-            <leftJoint>l_wheel_joint</leftJoint> <!-- 左轮 -->
-            <rightJoint>r_wheel_joint</rightJoint> <!-- 右轮 -->
+            <leftJoint>base_l_wheel_joint</leftJoint> <!-- 左轮 -->
+            <rightJoint>base_r_wheel_joint</rightJoint> <!-- 右轮 -->
             <wheelSeparation>${wheel_driving_between}</wheelSeparation> <!-- 车轮间距 -->
             <wheelDiameter>${wheel_driving_radius * 2}</wheelDiameter> <!-- 车轮直径 -->

File: src/model/xacro/gazebo/laser.xacro (robot description, xacro)
@@ -5,5 +5,5 @@
     <sensor type="ray" name="rplidar">
       <pose>0 0 0 0 0 0</pose>
-      <visualize>true</visualize>
+      <visualize>false</visualize>
       <update_rate>5.5</update_rate>
       <ray>

Commit message: modify gazebo

File: src/model/xacro/gazebo/base.xacro (robot description, xacro)
@@ -15,5 +15,5 @@
         <material>Gazebo/Yellow</material>
     </gazebo>
-        <!-- 传动实现:用于连接控制器与关节 -->
+        <!-- joint_transmission -->
     <xacro:macro name="joint_transmission" params="wheel_name">
         <!-- Transmission is important to link the joints and the controller -->
@@ -29,8 +29,8 @@
         </transmission>
     </xacro:macro>
-    <!-- 每一个驱动轮都需要配置传动装置 -->
+    <!-- settion transimision for driver wheel  -->
     <xacro:joint_transmission wheel_name="l_wheel"/>
     <xacro:joint_transmission wheel_name="r_wheel"/>
-    <!-- 控制器 -->
+    <!--differential controller -->
     <gazebo>
         <plugin name="differential_drive_controller" filename="libgazebo_ros_diff_drive.so">
@@ -39,21 +39,19 @@
             <robotNamespace>/</robotNamespace>
             <publishTf>1</publishTf>
-            <publishWheelJointState>falsee</publishWheelJointState>
+            <publishWheelJointState>false</publishWheelJointState>
             <alwaysOn>true</alwaysOn>
-            <updateRate>150.0</updateRate>
+            <updateRate>30.0</updateRate>
             <legacyMode>true</legacyMode>
-            <leftJoint>base_l_wheel_joint</leftJoint> <!-- 左轮 -->
-            <rightJoint>base_r_wheel_joint</rightJoint> <!-- 右轮 -->
-            <wheelSeparation>${wheel_driving_between}</wheelSeparation> <!-- 车轮间距 -->
-            <wheelDiameter>${wheel_driving_radius * 2}</wheelDiameter> <!-- 车轮直径 -->
+            <leftJoint>base_l_wheel_joint</leftJoint> <!-- left wheel -->
+            <rightJoint>base_r_wheel_joint</rightJoint> <!-- right wheel-->
+            <wheelSeparation>${wheel_driving_between}</wheelSeparation> <!-- distance of left and right wheel  -->
+            <wheelDiameter>${wheel_driving_radius * 2}</wheelDiameter> <!-- radius * 2 -->
             <broadcastTF>1</broadcastTF>
             <wheelTorque>30</wheelTorque>
             <wheelAcceleration>1.8</wheelAcceleration>
-            <commandTopic>cmd_vel</commandTopic> <!-- 运动控制话题 -->
+            <commandTopic>cmd_vel</commandTopic> <!-- topic for controller-->
             <odometryFrame>odom</odometryFrame>
-            <odometryTopic>odom</odometryTopic> <!-- 里程计话题 -->
-            <odometrySource>1</odometrySource>
-            <publishOdomTF>false</publishOdomTF>
-            <robotBaseFrame>base_footprint</robotBaseFrame> <!-- 根坐标系 -->
+            <odometryTopic>odom</odometryTopic> <!-- odmetry topic  -->
+            <robotBaseFrame>base_footprint</robotBaseFrame> <!-- base frame -->
         </plugin>
     </gazebo>

File: src/model/xacro/gazebo/laser.xacro (robot description, xacro)
@@ -1,4 +1,4 @@
 <robot name="laser" xmlns:xacro="http://wiki.ros.org/xacro">
-  <!-- 雷达 -->
+  <!-- laser -->
   <gazebo reference="laser_link">
     <material>Gazebo/Black</material>

File: src/model/xacro/link/base.xacro (robot description, xacro)
@@ -29,5 +29,5 @@
                 <origin xyz="0.0 0.0 0.0" rpy="${PI/2} 0.0 0.0" />
             </collision>
-            <xacro:cylinder_inertial_matrix m="2" r="${wheel_driving_radius}" h="${wheel_driving_width}"/>
+            <xacro:cylinder_inertial_matrix m="10" r="${wheel_driving_radius}" h="${wheel_driving_width}"/>
         </link>
         <joint name="base_${wheel_name}_joint" type="continuous">
@@ -94,5 +94,5 @@
             <origin xyz="0 0 0" rpy="0 0 0"/>
         </collision>
-        <xacro:cylinder_inertial_matrix m="4" r="${base_radius}" h="${base_length}"/>
+        <xacro:cylinder_inertial_matrix m="15" r="${base_radius}" h="${base_length}"/>
     </link>
     <joint name="base_link_joint" type="fixed">

File: src/model/xacro/link/laser.xacro (robot description, xacro)
@@ -2,8 +2,8 @@
     <xacro:property name="laser_length" value="0.025"/>
     <xacro:property name="laser_radius" value="0.025"/>
-<!--安装位置-->
+<!--laser position-->
     <xacro:property name="laser_joint_x" value="0"/>
     <xacro:property name="laser_joint_y" value="0"/>
-    <xacro:property name="laser_joint_z" value="0.14"/>
+    <xacro:property name="laser_joint_z" value="0.19"/>
     <link name="laser_link">
         <visual>
@@ -16,5 +16,5 @@
     </link>
     <joint name="lasesr_joint" type="fixed">
-        <parent link="base_link"/>
+        <parent link="base_footprint"/>
         <child link="laser_link"/>
         <origin xyz="${laser_joint_x} ${laser_joint_y} ${laser_joint_z}"/>

File: src/model/xacro/link/robot.xacro (robot description, xacro)
@@ -4,5 +4,5 @@
     <xacro:include filename="base.xacro"/>
     <xacro:include filename="laser.xacro"/>
-    <!--gazebo仿真-->
+    <!--gazebo-->
     <xacro:include filename="../gazebo/base.xacro"/>
     <xacro:include filename="../gazebo/laser.xacro"/>
